File: alexabase/alexakit.brd (EAGLE design)
At the start: 35.6 x 80 mm, 10 parts

Commit message: Update alexakit.
Routing:
- net GND: track 131.9 -> 124.6 mm
Changed lines of the file:
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@@
 <wire x1="9.6012" y1="64.77" x2="9.51" y2="64.87" width="0.1524" layer="1"/>
 <wire x1="7.7724" y1="62.7888" x2="7.79" y2="62.7" width="0.1524" layer="1"/>
-<wire x1="6.5532" y1="63.8556" x2="6.56" y2="63.72" width="0.1524" layer="1"/>
 <wire x1="5.6436" y1="64.9224" x2="5.75" y2="64.94" width="0.1524" layer="1"/>
 <wire x1="7.7724" y1="63.0936" x2="7.79" y2="63.15" width="0.1524" layer="1"/>
-<wire x1="6.7056" y1="63.7032" x2="6.56" y2="63.72" width="0.1524" layer="1"/>
 <wire x1="5.6388" y1="64.9224" x2="5.55" y2="64.94" width="0.1524" layer="1"/>
 <wire x1="9.4488" y1="64.9224" x2="9.51" y2="64.87" width="0.1524" layer="1"/>
@@
 <wire x1="6.35" y1="63.5" x2="6.35" y2="63.2" width="0.1524" layer="1"/>
 <wire x1="5.65" y1="63.2" x2="5.6388" y2="63.2" width="0.1524" layer="1"/>
-<wire x1="5.6388" y1="63.2" x2="5.6388" y2="64.9224" width="0.1524" layer="1"/>
 <wire x1="6.35" y1="63.2" x2="6.05" y2="63.2" width="0.1524" layer="1"/>
-<wire x1="6.05" y1="63.2" x2="6" y2="64.94" width="0.1524" layer="1"/>
 <wire x1="5.8386" y1="63.2" x2="5.65" y2="63.2" width="0.1524" layer="1"/>
-<wire x1="5.65" y1="63.2" x2="5.55" y2="64.94" width="0.1524" layer="1"/>
 <wire x1="5.65" y1="63.2" x2="4.7464" y2="63.2" width="0.1524" layer="1"/>
 <wire x1="4.7464" y1="63.2" x2="4.7464" y2="63.2364" width="0.1524" layer="1"/>
 <wire x1="6.05" y1="63.2" x2="5.8386" y2="63.2" width="0.1524" layer="1"/>
-<wire x1="5.8386" y1="63.2" x2="5.8386" y2="64.0636" width="0.1524" layer="1"/>
-<wire x1="5.8386" y1="64.0636" x2="4.840990625" y2="64.0636" width="0.1524" layer="1"/>
 <wire x1="6.35" y1="63.2" x2="6.4864" y2="63.2" width="0.1524" layer="1"/>
 <wire x1="6.4864" y1="63.2" x2="6.4864" y2="61.8964" width="0.1524" layer="1"/>
 <wire x1="5.75" y1="64.94" x2="6" y2="64.94" width="0.1524" layer="1"/>
-<wire x1="6.56" y1="63.72" x2="6.56" y2="63.5" width="0.1524" layer="1"/>
+<wire x1="6.2552" y1="63.42028125" x2="6.56" y2="63.5" width="0.1524" layer="1"/>
 <wire x1="6.56" y1="63.5" x2="6.35" y2="63.5" width="0.1524" layer="1"/>
 <wire x1="9.51" y1="64.87" x2="9.51" y2="68.58" width="0.1524" layer="1"/>
@@
 </polygon>
 <wire x1="4.840990625" y1="64.0636" x2="4.8244" y2="64.108" width="0.1524" layer="1"/>
+<wire x1="4.71" y1="64.1" x2="4.8244" y2="64.108" width="0" layer="19" extent="1-1"/>
+<wire x1="4.7464" y1="63.2364" x2="4.840990625" y2="64.0636" width="0" layer="19" extent="1-1"/>
 </signal>
 <signal name="13">
