File: analogmic/opamp.brd (EAGLE design)
At the start: 15.5 x 33.1 mm, 13 parts

Commit message: Update opamp.
Parts:
- moved OP1 2.21 mm to (7.60, 11.3)
Connections:
- removed net N$4: C3.1, R2.1
- net GND: now also C3.1, R2.1
Routing:
- net GND: track 64.8 -> 0.00 mm, vias 7 -> 0
- net 3V3: track 71.0 -> 33.7 mm, vias 0 -> 2
- net N$4: track 13.2 -> 0.00 mm
- net VCC: track 12.3 -> 17.0 mm
- net N$3: track 22.7 -> 20.5 mm
- net OUTPUT: track 37.0 -> 38.1 mm
- net N$5: track 24.4 -> 23.5 mm, vias 3 -> 2
