File: analogmic/opamp.sch (EAGLE design)
At the start: 12 parts

Commit message: Update opamp.
Parts:
- OP1: device FaBo-Opamp:OPA335 -> FaBo-Opamp:OPA344
Connections:
- removed net N$4: C3.1, R2.1
- net GND: now also C3.1, R2.1
Changed lines of the file:
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@@
 <part name="GND2" library="FaBo-Supply" deviceset="GND" device=""/>
 <part name="IN" library="FaBo-Template" deviceset="FABO_BRICK_3PIN" device="-S03B-PASK-2"/>
-<part name="OP1" library="FaBo-Opamp" deviceset="OPA335" device=""/>
 <part name="C2" library="FaBo-Capacitor" deviceset="CAPACITOR" device="-0603" value="4.7uF"/>
 <part name="R1" library="FaBo-Resistors" deviceset="RESISTOR" device="-0603" value="1.5K"/>
@@
 <part name="IC2" library="FaBo-Supply" deviceset="LP2985" device="-33DBV"/>
 <part name="VCC2" library="FaBo-Supply" deviceset="VCC" device=""/>
+<part name="GND6" library="FaBo-Supply" deviceset="GND" device=""/>
+<part name="OP1" library="FaBo-Opamp" deviceset="OPA344" device=""/>
 </parts>
 <sheets>
@@
 <attribute name="NAME" x="43.18" y="91.948" size="1.778" layer="95"/>
 </instance>
-<instance part="OP1" gate="G$1" x="137.16" y="127" smashed="yes">
-<attribute name="NAME" x="142.24" y="132.08" size="1.27" layer="95"/>
-</instance>
 <instance part="C2" gate="G$1" x="91.44" y="132.08" smashed="yes">
 <attribute name="NAME" x="89.154" y="134.366" size="1.4224" layer="95"/>
@@
 <instance part="VCC2" gate="G$1" x="205.74" y="165.1" smashed="yes">
 <attribute name="VALUE" x="204.47" y="168.656" size="1.778" layer="96"/>
+</instance>
+<instance part="GND6" gate="G$1" x="116.84" y="93.98" smashed="yes">
+<attribute name="VALUE" x="114.046" y="88.9" size="1.778" layer="96"/>
+</instance>
+<instance part="OP1" gate="G$1" x="137.16" y="127" smashed="yes">
+<attribute name="NAME" x="142.24" y="132.08" size="1.27" layer="95"/>
 </instance>
 </instances>
@@
 <segment>
 <wire x1="165.1" y1="170.18" x2="165.1" y2="162.56" width="0.1524" layer="91"/>
-<pinref part="OP1" gate="G$1" pin="OUT"/>
 <wire x1="165.1" y1="162.56" x2="165.1" y2="127" width="0.1524" layer="91"/>
 <wire x1="165.1" y1="127" x2="154.94" y2="127" width="0.1524" layer="91"/>
@@
 <junction x="165.1" y="127"/>
 <label x="177.8" y="127" size="1.778" layer="95"/>
+<pinref part="OP1" gate="G$1" pin="OUT"/>
 </segment>
 <segment>
@@
 </segment>
 <segment>
-<pinref part="OP1" gate="G$1" pin="V+"/>
 <pinref part="3V1" gate="G$1" pin="3V3"/>
 <wire x1="137.16" y1="139.7" x2="137.16" y2="152.4" width="0.1524" layer="91"/>
+<pinref part="OP1" gate="G$1" pin="V+"/>
 </segment>
 <segment>
@@
 </segment>
 <segment>
-<pinref part="OP1" gate="G$1" pin="V-"/>
 <wire x1="137.16" y1="114.3" x2="137.16" y2="104.14" width="0.1524" layer="91"/>
 <pinref part="GND1" gate="G$1" pin="GND"/>
+<pinref part="OP1" gate="G$1" pin="V-"/>
 </segment>
 <segment>
@@
 <pinref part="GND5" gate="G$1" pin="GND"/>
 </segment>
+<segment>
+<pinref part="C3" gate="G$1" pin="1"/>
+<wire x1="93.98" y1="104.14" x2="93.98" y2="99.06" width="0.1524" layer="91"/>
+<wire x1="93.98" y1="99.06" x2="116.84" y2="99.06" width="0.1524" layer="91"/>
+<wire x1="116.84" y1="99.06" x2="116.84" y2="106.68" width="0.1524" layer="91"/>
+<pinref part="R2" gate="G$1" pin="1"/>
+<wire x1="116.84" y1="99.06" x2="116.84" y2="93.98" width="0.1524" layer="91"/>
+<junction x="116.84" y="99.06"/>
+<pinref part="GND6" gate="G$1" pin="GND"/>
+</segment>
 </net>
 <net name="N$1" class="0">
@@
 <net name="N$3" class="0">
 <segment>
-<pinref part="OP1" gate="G$1" pin="+"/>
 <wire x1="124.46" y1="119.38" x2="116.84" y2="119.38" width="0.1524" layer="91"/>
 <pinref part="C3" gate="G$1" pin="2"/>
@@
 <pinref part="R3" gate="G$1" pin="1"/>
 <wire x1="116.84" y1="119.38" x2="116.84" y2="121.92" width="0.1524" layer="91"/>
-</segment>
-</net>
-<net name="N$4" class="0">
-<segment>
-<pinref part="C3" gate="G$1" pin="1"/>
-<wire x1="93.98" y1="104.14" x2="93.98" y2="99.06" width="0.1524" layer="91"/>
-<wire x1="93.98" y1="99.06" x2="116.84" y2="99.06" width="0.1524" layer="91"/>
-<wire x1="116.84" y1="99.06" x2="116.84" y2="106.68" width="0.1524" layer="91"/>
-<pinref part="R2" gate="G$1" pin="1"/>
+<pinref part="OP1" gate="G$1" pin="+"/>
 </segment>
 </net>
@@
 <segment>
 <pinref part="R1" gate="G$1" pin="2"/>
-<pinref part="OP1" gate="G$1" pin="-"/>
 <wire x1="124.46" y1="132.08" x2="121.92" y2="132.08" width="0.1524" layer="91"/>
 <wire x1="121.92" y1="132.08" x2="111.76" y2="132.08" width="0.1524" layer="91"/>
@@
 <pinref part="C4" gate="G$1" pin="1"/>
 <wire x1="121.92" y1="170.18" x2="137.16" y2="170.18" width="0.1524" layer="91"/>
-</segment>
-</net>
+<pinref part="OP1" gate="G$1" pin="-"/>
+</segment>
+</net>
