File: wroverdevkit/devkit.sch (EAGLE design)
At the start: 41 parts, among them IC1 FT231XQ, Q3 BSS138, Q4 BSS138, T1 TRANSISTORMMBT2222, T2 TRANSISTORMMBT2222, T3 TRANSISTORMMBT2222

Commit message: Update alexakit.
Parts:
- C6: value 100uf -> 100uF; device FaBo-Capacitor:CAPACITOR-0603_NARROW -> FaBo-Capacitor:CAPACITOR-1206
Connections:
- net DTR: now also T2.E, T3.E; no longer T2.C, T3.C
- net IO0: now also T2.C; no longer T2.E
- net IO2: now also T3.C; no longer T3.E
- net RXD: now also U$1.RXD0; no longer U$1.TXD0
- net TXD: now also U$1.TXD0; no longer U$1.RXD0

Commit message: Change TX and RX.
Connections:
- net RXD: now also IC1.TXD; no longer IC1.RXD
- net TXD: now also IC1.RXD; no longer IC1.TXD
Changed lines of the file:
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@@
-</segment>
-<segment>
-<pinref part="IC1" gate="G$1" pin="RXD"/>
-<wire x1="139.7" y1="53.34" x2="129.54" y2="53.34" width="0.1524" layer="91"/>
-<label x="134.62" y="53.34" size="1.778" layer="95"/>
 </segment>
 <segment>
@@
 <wire x1="238.76" y1="152.4" x2="248.92" y2="152.4" width="0.1524" layer="91"/>
 <label x="248.92" y="152.4" size="1.778" layer="95"/>
+</segment>
+<segment>
+<pinref part="IC1" gate="G$1" pin="TXD"/>
+<wire x1="139.7" y1="50.8" x2="129.54" y2="50.8" width="0.1524" layer="91"/>
+<label x="134.62" y="50.8" size="1.778" layer="95"/>
 </segment>
 </net>
@@
 </segment>
 <segment>
-<pinref part="IC1" gate="G$1" pin="TXD"/>
-<wire x1="139.7" y1="50.8" x2="129.54" y2="50.8" width="0.1524" layer="91"/>
-<label x="134.62" y="50.8" size="1.778" layer="95"/>
-</segment>
-<segment>
 <pinref part="U$1" gate="G$1" pin="TXD0"/>
 <wire x1="238.76" y1="154.94" x2="248.92" y2="154.94" width="0.1524" layer="91"/>
 <label x="248.92" y="154.94" size="1.778" layer="95"/>
 </segment>
+<segment>
+<pinref part="IC1" gate="G$1" pin="RXD"/>
+<wire x1="139.7" y1="53.34" x2="129.54" y2="53.34" width="0.1524" layer="91"/>
+<label x="134.62" y="53.34" size="1.778" layer="95"/>
+</segment>
 </net>

Commit message: devボード見直し
Parts:
- removed ., ..: (no value), pinhead:PINHD-1X19
- removed C10, C9: 27pf, FaBo-Capacitor:CAPACITOR-0603_NARROW
- removed C11, C12: 1nf, FaBo-Capacitor:CAPACITOR-0603_NARROW
- removed C13, C14: 1uF, FaBo-Capacitor:CAPACITOR-0603
- removed CY1: CRYSTALABS07, FaBo-Crystal:CRYSTALABS07
- removed EN: (no value), FaBo-Switch:TACT-SWITCH-SMD_KMR2
- removed F1: (no value), FaBo-Parts:POLYSWITCH
- removed Q3, Q4: BSS138, FaBo-etc:MOSFET-N-BSS138
- removed R10: 10K, FaBo-Resistors:RESISTOR-0603-NARROW
- removed R11, R12: 1K, FaBo-Resistors:RESISTOR-0603-NARROW
- removed R13, R14, R15: 100K, FaBo-Resistors:RESISTOR-0603-NARROW
- removed R5, R6: 5K, FaBo-Resistors:RESISTOR-0603-NARROW
- removed R8: 12K, FaBo-Resistors:RESISTOR-0603-NARROW
- removed R9: 470, FaBo-Resistors:RESISTOR-0603-NARROW
- removed T1, T2, T3: TRANSISTORMMBT2222, FaBo-Transistor:TRANSISTORMMBT2222
- removed U$1: ESP32-WROVER, FaBo-ESP32:ESP32-WROVER
- added C0: NP, component:CAPACITOR-M
- added CN1, CN2: (no value), component:PIN_1X19
- added D1: ESDA6V1BC6, component:ESDA6V1BC6
- added D2: (no value), component:DIODE_SCHOTTKY-RB161MM-20
- added FID1, FID2: FIDUCIAL-TOP, component:FIDUCIAL-TOP
- added LED1: (no value), component:LED-0603
- added LED2: (no value), component:HSMF-C16X
- added LOGO1: (no value), component:LOGO_FABO-M_BOTTOM
- added R3, R4: 1k, component:RESISTOR-0603
- added RESET: (no value), component:TACTILE-KMR2
- added U1: (no value), component:ESP32-WROVER-B
- added U2: TPS2065DBVR, component:TPS2065DBV
- added U3: BS138PS, component:BS138PS
- added X1: 32.768k, component:CRYSTAL-ABS07
- BOOT: device FaBo-Switch:TACT-SWITCH-SMD_KMR2 -> component:TACTILE-KMR2
- C1: value 47pF -> 0.1uF; device FaBo-Capacitor:CAPACITOR-0603_NARROW -> component:CAPACITOR-0603
- C2: value 47pF -> 0.01uF; device FaBo-Capacitor:CAPACITOR-0603_NARROW -> component:CAPACITOR-0603
- C3: value 0.1uF -> 1uF; device FaBo-Capacitor:CAPACITOR-0603_NARROW -> component:CAPACITOR-0603
- C4: value 4.7uF -> 1uF; device FaBo-Capacitor:CAPACITOR-0603_NARROW -> component:CAPACITOR-0603
- C5: value 0.1uF -> 4.3pF; device FaBo-Capacitor:CAPACITOR-0603_NARROW -> component:CAPACITOR-0603
- C6: value 100uF -> 4.3pF; device FaBo-Capacitor:CAPACITOR-1206 -> component:CAPACITOR-0603
- C7: value 1uf -> 10uF; device FaBo-Capacitor:CAPACITOR-0603_NARROW -> component:CAPACITOR-0603
- C8: value 0.1uf -> 0.1uF; device FaBo-Capacitor:CAPACITOR-0603_NARROW -> component:CAPACITOR-0603
- IC1: value FT231XQ -> ADP3338AKCZ-3.3; device FaBo-USB:FT231XQ -> component:ADP3338AKCZ
- IC2: value (none) -> FT231XQ; device FaBo-Supply:AP2112K-3.3TRG1 -> component:FT231XQ
- R1: value 27 -> 10k; device FaBo-Resistors:RESISTOR-0603-NARROW -> component:RESISTOR_ARRAY
- R2: value 27 -> 470; device FaBo-Resistors:RESISTOR-0603-NARROW -> component:RESISTOR-0603
- USB1: value (none) -> ZX62D-B-5PA8(30); device FaBo-USB:USB-MICRO_B_SMT_HIROSE -> component:USB-ZX62D
Connections:
- removed net CBUS1: IC1.CBUS1
- removed net CBUS2: IC1.CBUS2
- removed net IO16: ...12
- removed net IO17: ...11
- removed net N$1: R13.1, T1.B
- removed net N$11: Q4.G, R11.1
- removed net N$12: Q3.G, R12.1
- removed net N$2: R14.1, T2.B
- removed net N$29: U$1.NC@32
- removed net N$3: C2.2, R2.1, USB1.D-
- removed net N$34: U$1.NC@28
- removed net N$36: U$1.NC@27
- removed net N$4: C1.2, R1.1, USB1.D+
- removed net N$5: C11.2, EN.3, EN.4, R9.2
- removed net N$6: BOOT.3, BOOT.4, C12.2, R10.2, R11.2, R12.2
- removed net N$7: C5.2, IC1.3V3OUT, IC1.RESET, IC1.VCCIO
- removed net N$8: R15.1, T3.B
- removed net SVN: ..4, U$1.SENSOR_VN
- removed net SVP: ..3, U$1.SENSOR_VP
- removed net VBUS: F1.1, USB1.VBUS
- new net LED1K: LED1.CATHODE, R1G$4.1
- new net LED2K1: LED2.K2, R3.2
- new net LED2K2: LED2.K1, R4.2
- new net OUT5V: CN1.19, D2.K
- new net RXLED: IC2.CBUS1, R3.1
- new net SENSOR_VN: CN1.4, U1.SENSOR_VN
- new net SENSOR_VP: CN1.3, U1.SENSOR_VP
- new net TXLED: IC2.CBUS2, R4.1
- new net TXPIN: IC2.TXD, R2.1
- new net USBVBUS: D1.1, U2.EN, U2.IN, USB1.VBUS
- net 3V3: now also C0.2, C1.2, C4.2, C8.2, CN1.1, IC1.OUT-TAB, IC2.3V3OUT, IC2.RESET, IC2.VCC, IC2.VCCIO, LED1.ANODE, LED2.A1, LED2.A2, R1G$1.1, R1G$2.1, U1.3V3; no longer ..1, BOOT.1, BOOT.2, C14.2, C6.2, C7.2, IC2.VOUT, R5.2, R8.2, U$1.VDD33
- net 5V: now also C7.2, D2.A, IC1.IN, U2.OUT; no longer ..19, C13.2, C4.2, F1.2, IC1.VCC, IC2.EN, IC2.VIN
- net CLK: now also CN2.19, U1.CLK; no longer ...19, U$1.CLK
- net CMD: now also CN1.18, U1.CMD; no longer ..18, U$1.CMD
- net DTR: now also IC2.DTR, U3G$1.G, U3G$2.S; no longer IC1.DTR, R13.2, T2.E, T3.E
- net EN: now also C2.2, CN1.2, R1G$1.2, RESET.3, RESET.4, U1.EN, U3G$1.D; no longer ..2, C8.2, R8.1, R9.1, T1.C, U$1.EN
- net GND: now also BOOT.1, BOOT.2, C0.1, CN1.14, CN2.1, CN2.7, D1.2, D1.5, IC1.GND, IC2.GND@13, IC2.GND@21, IC2.GND@3, R1G$3.1, R1G$4.2, RESET.1, RESET.2, U1.GND@1, U1.GND@15, U1.GND@38, U1.GND@39, U2.GND; no longer ...1, ...7, ..14, C10.1, C11.1, C12.1, C13.1, C14.1, C9.1, EN.1, EN.2, IC1.GND@13, IC1.GND@21, IC1.GND@3, IC2.GND, Q3.S, Q4.S, R10.1, R6.1, U$1.GND@1, U$1.GND@15, U$1.GND@38, U$1.GND@39
- net IO0: now also BOOT.3, BOOT.4, CN2.14, R1G$2.2, U1.IO0, U3G$2.D; no longer ...14, Q4.D, R5.1, T2.C, U$1.IO0
- net IO12: now also CN1.13, U1.IO12; no longer ..13, U$1.IO12
- net IO13: now also CN1.15, U1.IO13; no longer ..15, U$1.IO13
- net IO14: now also CN1.12, U1.IO14; no longer ..12, U$1.IO14
- net IO15: now also CN2.16, U1.IO15; no longer ...16, U$1.IO15
- net IO18: now also CN2.9, U1.IO18; no longer ...9, U$1.IO18
- net IO19: now also CN2.8, U1.IO19; no longer ...8, U$1.IO19
- net IO2: now also CN2.15, R1G$3.2, U1.IO2; no longer ...15, Q3.D, R6.2, T3.C, U$1.IO2
- net IO21: now also CN2.6, U1.IO21; no longer ...6
- net IO22: now also CN2.3, U1.IO22; no longer ...3, U$1.IO21, U$1.IO22
- net IO23: now also CN2.2, U1.IO23; no longer ...2, U$1.IO23
- net IO25: now also CN1.9, U1.IO25; no longer ..9, U$1.IO25
- net IO26: now also CN1.10, U1.IO26; no longer ..10, U$1.IO26
- net IO27: now also CN1.11, U1.IO27; no longer ..11, U$1.IO27
- net IO32: now also C5.2, CN1.7, U1.IO32, X1.P$1; no longer ..7, C10.2, CY1.P$1, U$1.IO32
- net IO33: now also C6.2, CN1.8, U1.IO33, X1.P$2; no longer ..8, C9.2, CY1.P$2, U$1.IO33, U$1.IO35
- net IO34: now also CN1.5, U1.IO34; no longer ..5, U$1.IO34
- net IO35: now also CN1.6, U1.IO35; no longer ..6
- net IO4: now also CN2.13, U1.IO4; no longer ...13, U$1.IO4
- net IO5: now also CN2.10, U1.IO5; no longer ...10, U$1.IO5
- net RTS: now also IC2.RTS, U3G$1.S, U3G$2.G; no longer IC1.RTS, R14.2, R15.2, T1.E
- net RXD: now also CN2.5, IC2.RXD, U1.RXD0; no longer ...4, IC1.TXD, U$1.RXD0
- net SD0: now also CN2.18, U1.SD0; no longer ...18, U$1.SD0
- net SD1: now also CN2.17, U1.SD1; no longer ...17, U$1.SD1
- net SD2: now also CN1.16, U1.SD2; no longer ..16, U$1.SD2
- net SD3: now also CN1.17, U1.SD3; no longer ..17, U$1.SD3
- net TXD: now also CN2.4, R2.2, U1.TXD0; no longer ...5, IC1.RXD, U$1.TXD0
- net USBDM: now also D1.3, IC2.USBDM, USB1.D-; no longer IC1.USBDM, R2.2
- net USBDP: now also D1.4, IC2.USBDP, USB1.D+; no longer IC1.USBDP, R1.2
Other:
- note added: "0.3"
- note added: "USB VBUS SOURCE"
- moved on the sheet: BOOT, C1, C2, C3, C4, C5, C6, C7, C8, R1G$1, R2

Commit message: fix route
Connections:
- net RXD: now also R2.2; no longer IC2.RXD
- net TXD: now also IC2.RXD; no longer R2.2
Other:
- note added: "0.4"
- note removed: "0.3"
Changed lines of the file:
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@@
 <sheet>
 <plain>
-<text x="246.38" y="20.32" size="2.54" layer="94" align="bottom-center">0.3</text>
+<text x="246.38" y="20.32" size="2.54" layer="94" align="bottom-center">0.4</text>
 <text x="208.28" y="99.06" size="1.27" layer="97">USB VBUS SOURCE</text>
 </plain>
@@
 </segment>
 <segment>
-<pinref part="R2" gate="G$1" pin="2"/>
-<wire x1="157.48" y1="53.34" x2="154.94" y2="53.34" width="0.1524" layer="91"/>
-<label x="157.48" y="53.34" size="1.27" layer="95" xref="yes"/>
-</segment>
-<segment>
 <wire x1="233.68" y1="81.28" x2="238.76" y2="81.28" width="0.1524" layer="91"/>
 <label x="233.68" y="81.28" size="1.27" layer="95" rot="R180" xref="yes"/>
 <pinref part="CN2" gate="G$1" pin="4"/>
+</segment>
+<segment>
+<pinref part="IC2" gate="G$1" pin="RXD"/>
+<wire x1="160.02" y1="50.8" x2="144.78" y2="50.8" width="0.1524" layer="91"/>
+<label x="160.02" y="50.8" size="1.27" layer="95" xref="yes"/>
 </segment>
 </net>
@@
 </segment>
 <segment>
-<pinref part="IC2" gate="G$1" pin="RXD"/>
-<wire x1="157.48" y1="50.8" x2="144.78" y2="50.8" width="0.1524" layer="91"/>
-<label x="157.48" y="50.8" size="1.27" layer="95" xref="yes"/>
-</segment>
-<segment>
 <wire x1="233.68" y1="78.74" x2="238.76" y2="78.74" width="0.1524" layer="91"/>
 <label x="233.68" y="78.74" size="1.27" layer="95" rot="R180" xref="yes"/>
 <pinref part="CN2" gate="G$1" pin="5"/>
 </segment>
+<segment>
+<pinref part="R2" gate="G$1" pin="2"/>
+<wire x1="160.02" y1="53.34" x2="154.94" y2="53.34" width="0.1524" layer="91"/>
+<label x="160.02" y="53.34" size="1.27" layer="95" xref="yes"/>
+</segment>
 </net>
