File: SensorHub/sensorHubRev4.sch (EAGLE design)
At the start: 57 parts, among them IC1 ADP3338AKCZ-3.3, IC2 FT231XQ, U2 TPS2065DBVR, U3 BS138PS, X1 32.768k, X2 332-02, X3 332-02

Commit message: SensorHubRev4Update
Addtion i2C EMI Filter Add
Parts:
- removed U$3: RUBYCONWXA1000UF/10V, FaBo-Capacitor:RUBYCONWXA1000UF/10V
- added C10: DNP, component:CAPACITOR-0603
- added C11, C9: 10uF, FaBo-Capacitor:CAPACITOR-0603_NARROW
- added C13, C14, C15, C16: 33pF, FaBo-Capacitor:CAPACITOR-0603_NARROW
- added C17: 0.1uF, component:CAPACITOR-0603
- added L1, L2, L3, L4: BLM18EG221SN1, FaBo-Inductor:INDUCTOR-0603
- added SJ1, SJ2: (no value), jumper:SJ
- added TP7: TPB1,27, testpad:TPB1,27
- C4: value 1uF -> 2.2uF
- R8, R9: value 1k -> 22
Connections:
- new net GNDIO: C11.1, C15.1, C16.1, C17.1, J1.GND, J10.GND, J11.GND, J12.GND, J2.GND, J3.GND, J4.GND, J5.GND, J6.GND, J7.GND, J8.GND, J9.GND, L4.2, SJ2.2, U$2.-
- new net N$7: C13.2, L2.1, R8.2
- new net N$8: C14.2, L3.1, R9.2
- new net VCCIO: C11.2, C17.2, J1.VCC, J10.VCC, J11.VCC, J12.VCC, J2.VCC, J3.VCC, J4.VCC, J5.VCC, J6.VCC, J7.VCC, J8.VCC, J9.VCC, L1.2, SJ1.1, TP7.TP, U$2.+
- net 3V3: now also C10.2, C9.2, L1.1, SJ1.2; no longer J1.VCC, J10.VCC, J11.VCC, J12.VCC, J2.VCC, J3.VCC, J4.VCC, J5.VCC, J6.VCC, J7.VCC, J8.VCC, J9.VCC, U$2.+, U$3.+
- net GND: now also C10.1, C13.1, C14.1, C9.1, L4.1, SJ2.1; no longer J1.GND, J10.GND, J11.GND, J12.GND, J2.GND, J3.GND, J4.GND, J5.GND, J6.GND, J7.GND, J8.GND, J9.GND, U$2.-, U$3.-
- net SCL: now also C16.2, L3.2; no longer R9.2
- net SDA: now also C15.2, L2.2; no longer R8.2
Other:
- moved on the sheet: BOOT, C3, C4, C5, C6, IC1, J6, POW, R10, R11, R12, R1G$3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
