File: SensorHub/sensorHubRev6.brd (EAGLE design)
At the start: 80 x 80 mm, 71 parts, among them IC1 ADP3338AKCZ-3.3, IC2 FT231XQ, U2 TPS2065DBVR, U3 BS138PS, X1 32.768k, X2 332-02, X3 332-02

Commit message: Revsionup to 6
Parts:
- removed C10: DNP, component:EIA0603
- removed C11: 10uF, FaBo-Capacitor:0603-NARROW
- removed C13, C14, C15, C16: 33pF, FaBo-Capacitor:0603-NARROW
- removed C17: 0.1uF, component:EIA0603
- removed L1, L2, L3, L4: BLM18EG221SN1, FaBo-Inductor:0603
- removed SJ1, SJ2: (no value), jumper:SJ
- removed U$2: RUBYCONWXA1000UF/10V, FaBo-Capacitor:ALUMINUM10*9
- added JMP1, JMP2: 0R-JUMPA, jump-0r-smd:A0R-JMP
- added R13: 10k, component:EIA0603
- added R14, R15: 22, component:EIA0603
- added R16: DNP, component:EIA0603
- added U5: LTC4313, FaBo-LevelTranslator:LTC4313
- C9: value 10uF -> 0.01uF; device FaBo-Capacitor:0603-NARROW -> component:EIA0603
- R6, R7: value 2.2k -> 2.2K
- R8, R9: value 22 -> 2k
- moved TP5 42.5 mm to (31.3, 29.4)
- moved R9 26.0 mm to (60.2, 37.0)
- moved R8 16.7 mm to (60.0, 39.9)
- moved TP7 15.4 mm to (53.0, 37.9)
- moved R7 12.0 mm to (56.7, 52.9)
- moved C9 10.6 mm to (62.0, 45.8), turned to 180 degrees
- moved POW 8.40 mm to (40.5, 38.5)
- moved TP2 6.95 mm to (51.1, 44.0)
- moved R6 4.96 mm to (56.8, 50.1)
- moved TP1 3.81 mm to (59.8, 29.9)
- moved J7 2.01 mm to (26.4, 11.7), turned to 154 degrees
- moved J2 1.88 mm to (66.7, 56.7), turned to 302 degrees
- moved J6 1.75 mm to (53.5, 11.7), turned to 206 degrees
- moved RESET 1.30 mm to (24.1, 32.8)
- moved J9 1.26 mm to (9.83, 31.3), turned to 106 degrees
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Connections:
- removed net GNDIO: C11.1, C15.1, C16.1, C17.1, J1.GND, J10.GND, J11.GND, J12.GND, J2.GND, J3.GND, J4.GND, J5.GND, J6.GND, J7.GND, J8.GND, J9.GND, L4.2, SJ2.2, U$2.MINUS
- removed net VCCIO: C11.2, C17.2, J1.VCC, J10.VCC, J11.VCC, J12.VCC, J2.VCC, J3.VCC, J4.VCC, J5.VCC, J6.VCC, J7.VCC, J8.VCC, J9.VCC, L1.2, SJ1.1, TP7.TP, U$2.PLUS
- new net N$10: R14.2, R6.2, U1.33
- new net N$11: R16.1, TP7.TP
- new net N$12: R15.2, R7.2, U1.36
- new net N$9: JMP2.2, R15.1
- net 3V3: now also R6.1, R7.1, U5.P$1, U5.P$8; no longer C10.2, L1.1, R6.2, R7.2, SJ1.2
- net 5V: now also J1.VCC, J10.VCC, J11.VCC, J12.VCC, J2.VCC, J3.VCC, J4.VCC, J5.VCC, J6.VCC, J7.VCC, J8.VCC, J9.VCC, R13.2, R8.2, R9.2
- net GND: now also J1.GND, J10.GND, J11.GND, J12.GND, J2.GND, J3.GND, J4.GND, J5.GND, J6.GND, J7.GND, J8.GND, J9.GND, U5.P$4; no longer C10.1, C13.1, C14.1, L4.1, SJ2.1
- net N$5: now also JMP1.3, U5.P$6; no longer R6.1, R8.1, U1.33
- net N$6: now also JMP2.3, U5.P$3; no longer R7.1, R9.1, U1.36
- net N$7: now also R13.1, R16.2, U5.P$5; no longer C13.2, L2.1, R8.2
- net N$8: now also JMP1.2, R14.1; no longer C14.2, L3.1, R9.2
- net SCL: now also JMP2.1, R8.1, U5.P$2; no longer C16.2, L3.2
- net SDA: now also JMP1.1, R9.1, U5.P$7; no longer C15.2, L2.2
Routing:
- net GNDIO: track 331.3 -> 0.00 mm
- net 5V: track 10.8 -> 308.8 mm, vias 0 -> 1
- net VCCIO: track 238.2 -> 0.00 mm
- net SDA: track 252.4 -> 295.0 mm, vias 5 -> 11
- net N$10: track 0.00 -> 27.3 mm, vias 0 -> 2
- net N$12: track 0.00 -> 24.1 mm
- net 3V3: track 219.3 -> 203.0 mm, vias 8 -> 9
- net GND: track 678.1 -> 667.7 mm, vias 113 -> 79
- net LED1K: track 8.76 -> 16.2 mm
- net N$8: track 4.60 -> 11.1 mm, vias 0 -> 1
- net N$9: track 0.00 -> 5.59 mm, vias 0 -> 1
- net IO33: track 9.98 -> 12.2 mm
- net N$11: track 0.00 -> 2.00 mm
- net N$7: track 6.87 -> 8.72 mm
- net N$6: track 9.95 -> 8.49 mm, vias 0 -> 1
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Other:
- board text added: "Rev.0.6"
- board text removed: "Rev.0.4"
